Commit message: update: ur10 tasks

File: urdf/grippers/Barrett/Barrett.urdf (robot description, URDF)
Before this commit: robot Barrett, 27 links, 26 joints
Joints:
- removed joint a_link1_link2_joint
- removed joint a_link2_link3_joint
- removed joint a_palm_link1_joint
- removed joint b_link1_link2_joint
- removed joint b_link2_link3_joint
- removed joint b_palm_link1_joint
- removed joint c_link2_link3_joint
- removed joint c_palm_link2_joint_0
- added joint bh_j11_joint: type revolute, parent palm, child a_link1_joint, origin xyz=0.02500000 0.00000000 -0.00100000 rpy=0.00000000 3.14159265 0.00000000, axis 0.00000000 0.00000000 1.00000000, limit lower=0.0 upper=3.14159265359 effort=50.00000000 velocity=0.52333333
- added joint bh_j12_joint: type revolute, parent a_link1, child a_link2_joint, origin xyz=0.00000000 0.00000000 0.00000000 rpy=0.00000000 0.00000000 0.00000000, axis 0.00000000 0.00000000 1.00000000, limit lower=0.0 upper=2.51327412287 effort=2.50000000 velocity=0.52333333
- added joint bh_j13_joint: type revolute, parent a_link2, child a_link3_joint, origin xyz=0.00000000 0.00000000 0.00000000 rpy=0.00000000 0.00000000 0.00000000, axis 0.00000000 0.00000000 0.33333333, limit lower=0.0 upper=2.51327412287 effort=2.50000000 velocity=0.52333333
- added joint bh_j21_joint: type revolute, parent palm, child b_link1_joint, origin xyz=-0.02500000 0.00000000 -0.00100000 rpy=0.00000000 0.00000000 0.00000000, axis 0.00000000 0.00000000 1.00000000, limit lower=0.0 upper=3.14159265359 effort=50.00000000 velocity=0.52333333
- added joint bh_j22_joint: type revolute, parent b_link1, child b_link2_joint, origin xyz=0.00000000 0.00000000 0.00000000 rpy=0.00000000 0.00000000 0.00000000, axis 0.00000000 0.00000000 1.00000000, limit lower=0.0 upper=2.51327412287 effort=2.50000000 velocity=0.52333333
- added joint bh_j23_joint: type revolute, parent b_link2, child b_link3_joint, origin xyz=0.00000000 0.00000000 0.00000000 rpy=0.00000000 0.00000000 0.00000000, axis 0.00000000 0.00000000 0.33333333, limit lower=0.0 upper=2.51327412287 effort=2.50000000 velocity=0.52333333
- added joint bh_j32_joint: type revolute, parent palm, child c_link2_joint_0, origin xyz=0.00000000 -0.05000000 -0.00100000 rpy=0.00000000 -1.57079633 0, axis 0.00000000 0.00000000 1.00000000, limit lower=0.0 upper=2.51327412287 effort=5.00000000 velocity=0.52333333
- added joint bh_j33_joint: type revolute, parent c_link2, child c_link3_joint, origin xyz=0.00000000 0.00000000 0.00000000 rpy=0.00000000 0.00000000 0.00000000, axis 0.00000000 0.00000000 0.33333333, limit lower=0.0 upper=2.51327412287 effort=5.00000000 velocity=0.52333333
